File: KAC12040_sfe_v0.1.brd (EAGLE design)
At the start: 101.6 x 57.1 mm, 2 parts

Commit message: Differential net names for LVDS
Connections:
- net N$10 renamed C$2_N
- net N$11 renamed L0$2_P
- net N$12 renamed L0$2_N
- net N$13 renamed L1$2_P
- net N$14 renamed L1$2_N
- net N$15 renamed L2$2_P
- net N$16 renamed L2$2_N
- net N$17 renamed L3$2_P
- net N$18 renamed L3$2_N
- net N$19 renamed L4$2_P
- net N$20 renamed L4$2_N
- net N$21 renamed L5$2_P
- net N$22 renamed L5$2_N
- net N$23 renamed L6$2_P
- net N$24 renamed L6$2_N
- net N$25 renamed L6$0_N
- net N$26 renamed L6$0_P
- net N$27 renamed L5$0_N
- net N$28 renamed L5$0_P
- net N$29 renamed L4$0_N
- net N$30 renamed L4$0_P
- net N$31 renamed L3$0_N
- net N$32 renamed L3$0_P
- net N$33 renamed L2$3_N
- net N$34 renamed L2$3_P
- net N$35 renamed L1$3_N
- net N$36 renamed L1$3_P
- net N$37 renamed L0$3_N
- net N$38 renamed L0$3_P
- net N$39 renamed C$3_N
- net N$40 renamed C$3_P
- net N$41 renamed L3$3_P
- net N$42 renamed L3$3_N
- net N$43 renamed L4$3_P
- net N$44 renamed L4$3_N
- net N$45 renamed L5$3_P
- net N$46 renamed L5$3_N
- net N$47 renamed L6$3_P
- net N$48 renamed L6$3_N
- net N$49 renamed C$1_P
- net N$5 renamed L1$0_P
- net N$50 renamed C$1_N
- net N$51 renamed L0$1_P
- net N$52 renamed L0$1_N
- net N$53 renamed L1$1_P
- net N$54 renamed L1$1_N
- net N$55 renamed L2$1_P
- net N$56 renamed L2$1_N
- net N$57 renamed L3$1_P
- net N$58 renamed L3$1_N
- net N$59 renamed L4$1_P
- net N$6 renamed L1$0_N
- net N$60 renamed L4$1_N
- net N$61 renamed L5$1_P
- net N$62 renamed L5$1_N
- net N$63 renamed L6$1_P
- net N$64 renamed L6$1_N
- net N$7 renamed L2$0_P
- net N$8 renamed L2$0_N
- net N$9 renamed C$2_P
