File: KAC12040_sfe_v0.1.sch (EAGLE design)
At the start: 2 parts

Commit message: Differential net names for LVDS
Connections:
- net N$10 renamed C$2_N
- net N$11 renamed L0$2_P
- net N$12 renamed L0$2_N
- net N$13 renamed L1$2_P
- net N$14 renamed L1$2_N
- net N$15 renamed L2$2_P
- net N$16 renamed L2$2_N
- net N$17 renamed L3$2_P
- net N$18 renamed L3$2_N
- net N$19 renamed L4$2_P
- net N$20 renamed L4$2_N
- net N$21 renamed L5$2_P
- net N$22 renamed L5$2_N
- net N$23 renamed L6$2_P
- net N$24 renamed L6$2_N
- net N$25 renamed L6$0_N
- net N$26 renamed L6$0_P
- net N$27 renamed L5$0_N
- net N$28 renamed L5$0_P
- net N$29 renamed L4$0_N
- net N$30 renamed L4$0_P
- net N$31 renamed L3$0_N
- net N$32 renamed L3$0_P
- net N$33 renamed L2$3_N
- net N$34 renamed L2$3_P
- net N$35 renamed L1$3_N
- net N$36 renamed L1$3_P
- net N$37 renamed L0$3_N
- net N$38 renamed L0$3_P
- net N$39 renamed C$3_N
- net N$40 renamed C$3_P
- net N$41 renamed L3$3_P
- net N$42 renamed L3$3_N
- net N$43 renamed L4$3_P
- net N$44 renamed L4$3_N
- net N$45 renamed L5$3_P
- net N$46 renamed L5$3_N
- net N$47 renamed L6$3_P
- net N$48 renamed L6$3_N
- net N$49 renamed C$1_P
- net N$5 renamed L1$0_P
- net N$50 renamed C$1_N
- net N$51 renamed L0$1_P
- net N$52 renamed L0$1_N
- net N$53 renamed L1$1_P
- net N$54 renamed L1$1_N
- net N$55 renamed L2$1_P
- net N$56 renamed L2$1_N
- net N$57 renamed L3$1_P
- net N$58 renamed L3$1_N
- net N$59 renamed L4$1_P
- net N$6 renamed L1$0_N
- net N$60 renamed L4$1_N
- net N$61 renamed L5$1_P
- net N$62 renamed L5$1_N
- net N$63 renamed L6$1_P
- net N$64 renamed L6$1_N
- net N$7 renamed L2$0_P
- net N$8 renamed L2$0_N
- net N$9 renamed C$2_P
Changed lines of the file:
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@@
 </segment>
 </net>
-<net name="N$5" class="0">
+<net name="L1$0_P" class="0">
 <segment>
 <pinref part="ZED1" gate="JX1_01" pin="_P"/>
@@
 </segment>
 </net>
-<net name="N$6" class="0">
+<net name="L1$0_N" class="0">
 <segment>
 <pinref part="ZED1" gate="JX1_01" pin="_N"/>
@@
 </segment>
 </net>
-<net name="N$7" class="0">
+<net name="L2$0_P" class="0">
 <segment>
 <pinref part="ZED1" gate="JX1_02" pin="_P"/>
@@
 </segment>
 </net>
-<net name="N$8" class="0">
+<net name="L2$0_N" class="0">
 <segment>
 <pinref part="ZED1" gate="JX1_02" pin="_N"/>
@@
 </segment>
 </net>
-<net name="N$9" class="0">
+<net name="C$2_P" class="0">
 <segment>
 <pinref part="ZED1" gate="JX1_11" pin="_P"/>
@@
 </segment>
 </net>
-<net name="N$10" class="0">
+<net name="C$2_N" class="0">
 <segment>
 <pinref part="ZED1" gate="JX1_11" pin="_N"/>
@@
 </segment>
 </net>
-<net name="N$11" class="0">
+<net name="L0$2_P" class="0">
 <segment>
 <pinref part="ZED1" gate="JX1_08" pin="_P"/>
@@
 </segment>
 </net>
-<net name="N$12" class="0">
+<net name="L0$2_N" class="0">
 <segment>
 <pinref part="ZED1" gate="JX1_08" pin="_N"/>
@@
 </segment>
 </net>
-<net name="N$13" class="0">
+<net name="L1$2_P" class="0">
 <segment>
 <pinref part="ZED1" gate="JX1_09" pin="_P"/>
@@
 </segment>
 </net>
-<net name="N$14" class="0">
+<net name="L1$2_N" class="0">
 <segment>
 <pinref part="ZED1" gate="JX1_09" pin="_N"/>
@@
 </segment>
 </net>
-<net name="N$15" class="0">
+<net name="L2$2_P" class="0">
 <segment>
 <pinref part="ZED1" gate="JX1_14" pin="_P"/>
@@
 </segment>
 </net>
-<net name="N$16" class="0">
+<net name="L2$2_N" class="0">
 <segment>
 <pinref part="ZED1" gate="JX1_14" pin="_N"/>
@@
 </segment>
 </net>
-<net name="N$17" class="0">
+<net name="L3$2_P" class="0">
 <segment>
 <pinref part="U$1" gate="_BANK2" pin="LVDS_3_P"/>
@@
 </segment>
 </net>
-<net name="N$18" class="0">
+<net name="L3$2_N" class="0">
 <segment>
 <pinref part="U$1" gate="_BANK2" pin="LVDS_3_N"/>
@@
 </segment>
 </net>
-<net name="N$19" class="0">
+<net name="L4$2_P" class="0">
 <segment>
 <pinref part="U$1" gate="_BANK2" pin="LVDS_4_P"/>
@@
 </segment>
 </net>
-<net name="N$20" class="0">
+<net name="L4$2_N" class="0">
 <segment>
 <pinref part="U$1" gate="_BANK2" pin="LVDS_4_N"/>
@@
 </segment>
 </net>
-<net name="N$21" class="0">
+<net name="L5$2_P" class="0">
 <segment>
 <pinref part="U$1" gate="_BANK2" pin="LVDS_5_P"/>
@@
 </segment>
 </net>
-<net name="N$22" class="0">
+<net name="L5$2_N" class="0">
 <segment>
 <pinref part="U$1" gate="_BANK2" pin="LVDS_5_N"/>
@@
 </segment>
 </net>
-<net name="N$23" class="0">
+<net name="L6$2_P" class="0">
 <segment>
 <pinref part="U$1" gate="_BANK2" pin="LVDS_6_P"/>
@@
 </segment>
 </net>
-<net name="N$24" class="0">
+<net name="L6$2_N" class="0">
 <segment>
 <pinref part="U$1" gate="_BANK2" pin="LVDS_6_N"/>
@@
 </segment>
 </net>
-<net name="N$25" class="0">
+<net name="L6$0_N" class="0">
 <segment>
 <pinref part="U$1" gate="_BANK0" pin="LVDS_6_N"/>
@@
 </segment>
 </net>
-<net name="N$26" class="0">
+<net name="L6$0_P" class="0">
 <segment>
 <pinref part="U$1" gate="_BANK0" pin="LVDS_6_P"/>
@@
 </segment>
 </net>
-<net name="N$27" class="0">
+<net name="L5$0_N" class="0">
 <segment>
 <pinref part="U$1" gate="_BANK0" pin="LVDS_5_N"/>
@@
 </segment>
 </net>
-<net name="N$28" class="0">
+<net name="L5$0_P" class="0">
 <segment>
 <pinref part="U$1" gate="_BANK0" pin="LVDS_5_P"/>
@@
 </segment>
 </net>
-<net name="N$29" class="0">
+<net name="L4$0_N" class="0">
 <segment>
 <pinref part="U$1" gate="_BANK0" pin="LVDS_4_N"/>
@@
 </segment>
 </net>
-<net name="N$30" class="0">
+<net name="L4$0_P" class="0">
 <segment>
 <pinref part="U$1" gate="_BANK0" pin="LVDS_4_P"/>
@@
 </segment>
 </net>
-<net name="N$31" class="0">
+<net name="L3$0_N" class="0">
 <segment>
 <pinref part="U$1" gate="_BANK0" pin="LVDS_3_N"/>
@@
 </segment>
 </net>
-<net name="N$32" class="0">
+<net name="L3$0_P" class="0">
 <segment>
 <pinref part="U$1" gate="_BANK0" pin="LVDS_3_P"/>
@@
 </segment>
 </net>
-<net name="N$33" class="0">
+<net name="L2$3_N" class="0">
 <segment>
 <pinref part="ZED1" gate="JX2_14" pin="_N"/>
@@
 </segment>
 </net>
-<net name="N$34" class="0">
+<net name="L2$3_P" class="0">
 <segment>
 <pinref part="ZED1" gate="JX2_14" pin="_P"/>
@@
 </segment>
 </net>
-<net name="N$35" class="0">
+<net name="L1$3_N" class="0">
 <segment>
 <pinref part="ZED1" gate="JX2_09" pin="_N"/>
@@
 </segment>
 </net>
-<net name="N$36" class="0">
+<net name="L1$3_P" class="0">
 <segment>
 <pinref part="ZED1" gate="JX2_09" pin="_P"/>
@@
 </segment>
 </net>
-<net name="N$37" class="0">
+<net name="L0$3_N" class="0">
 <segment>
 <pinref part="ZED1" gate="JX2_08" pin="_N"/>
@@
 </segment>
 </net>
-<net name="N$38" class="0">
+<net name="L0$3_P" class="0">
 <segment>
 <pinref part="ZED1" gate="JX2_08" pin="_P"/>
@@
 </segment>
 </net>
-<net name="N$39" class="0">
+<net name="C$3_N" class="0">
 <segment>
 <pinref part="ZED1" gate="JX2_11" pin="_N"/>
@@
 </segment>
 </net>
-<net name="N$40" class="0">
+<net name="C$3_P" class="0">
 <segment>
 <pinref part="ZED1" gate="JX2_11" pin="_P"/>
@@
 </segment>
 </net>
-<net name="N$41" class="0">
+<net name="L3$3_P" class="0">
 <segment>
 <pinref part="U$1" gate="_BANK3" pin="LVDS_3_P"/>
@@
 </segment>
 </net>
-<net name="N$42" class="0">
+<net name="L3$3_N" class="0">
 <segment>
 <pinref part="U$1" gate="_BANK3" pin="LVDS_3_N"/>
@@
 </segment>
 </net>
-<net name="N$43" class="0">
+<net name="L4$3_P" class="0">
 <segment>
 <pinref part="U$1" gate="_BANK3" pin="LVDS_4_P"/>
@@
 </segment>
 </net>
-<net name="N$44" class="0">
+<net name="L4$3_N" class="0">
 <segment>
 <pinref part="U$1" gate="_BANK3" pin="LVDS_4_N"/>
@@
 </segment>
 </net>
-<net name="N$45" class="0">
+<net name="L5$3_P" class="0">
 <segment>
 <pinref part="U$1" gate="_BANK3" pin="LVDS_5_P"/>
@@
 </segment>
 </net>
-<net name="N$46" class="0">
+<net name="L5$3_N" class="0">
 <segment>
 <pinref part="U$1" gate="_BANK3" pin="LVDS_5_N"/>
@@
 </segment>
 </net>
-<net name="N$47" class="0">
+<net name="L6$3_P" class="0">
 <segment>
 <pinref part="U$1" gate="_BANK3" pin="LVDS_6_P"/>
@@
 </segment>
 </net>
-<net name="N$48" class="0">
+<net name="L6$3_N" class="0">
 <segment>
 <pinref part="U$1" gate="_BANK3" pin="LVDS_6_N"/>
@@
 </segment>
 </net>
-<net name="N$49" class="0">
+<net name="C$1_P" class="0">
 <segment>
 <pinref part="ZED1" gate="JX2_10" pin="_P"/>
@@
 </segment>
 </net>
-<net name="N$50" class="0">
+<net name="C$1_N" class="0">
 <segment>
 <pinref part="ZED1" gate="JX2_10" pin="_N"/>
@@
 </segment>
 </net>
-<net name="N$51" class="0">
+<net name="L0$1_P" class="0">
 <segment>
 <pinref part="ZED1" gate="JX2_00" pin="_P"/>
@@
 </segment>
 </net>
-<net name="N$52" class="0">
+<net name="L0$1_N" class="0">
 <segment>
 <pinref part="ZED1" gate="JX2_00" pin="_N"/>
@@
 </segment>
 </net>
-<net name="N$53" class="0">
+<net name="L1$1_P" class="0">
 <segment>
 <pinref part="ZED1" gate="JX2_01" pin="_P"/>
@@
 </segment>
 </net>
-<net name="N$54" class="0">
+<net name="L1$1_N" class="0">
 <segment>
 <pinref part="ZED1" gate="JX2_01" pin="_N"/>
@@
 </segment>
 </net>
-<net name="N$55" class="0">
+<net name="L2$1_P" class="0">
 <segment>
 <pinref part="ZED1" gate="JX2_02" pin="_P"/>
@@
 </segment>
 </net>
-<net name="N$56" class="0">
+<net name="L2$1_N" class="0">
 <segment>
 <pinref part="ZED1" gate="JX2_02" pin="_N"/>
@@
 </segment>
 </net>
-<net name="N$57" class="0">
+<net name="L3$1_P" class="0">
 <segment>
 <pinref part="U$1" gate="_BANK1" pin="LVDS_3_P"/>
@@
 </segment>
 </net>
-<net name="N$58" class="0">
+<net name="L3$1_N" class="0">
 <segment>
 <pinref part="U$1" gate="_BANK1" pin="LVDS_3_N"/>
@@
 </segment>
 </net>
-<net name="N$59" class="0">
+<net name="L4$1_P" class="0">
 <segment>
 <pinref part="U$1" gate="_BANK1" pin="LVDS_4_P"/>
@@
 </segment>
 </net>
-<net name="N$60" class="0">
+<net name="L4$1_N" class="0">
 <segment>
 <pinref part="U$1" gate="_BANK1" pin="LVDS_4_N"/>
@@
 </segment>
 </net>
-<net name="N$61" class="0">
+<net name="L5$1_P" class="0">
 <segment>
 <pinref part="U$1" gate="_BANK1" pin="LVDS_5_P"/>
@@
 </segment>
 </net>
-<net name="N$62" class="0">
+<net name="L5$1_N" class="0">
 <segment>
 <pinref part="U$1" gate="_BANK1" pin="LVDS_5_N"/>
@@
 </segment>
 </net>
-<net name="N$63" class="0">
+<net name="L6$1_P" class="0">
 <segment>
 <pinref part="U$1" gate="_BANK1" pin="LVDS_6_P"/>
@@
 </segment>
 </net>
-<net name="N$64" class="0">
+<net name="L6$1_N" class="0">
 <segment>
 <pinref part="U$1" gate="_BANK1" pin="LVDS_6_N"/>
