File: KAC12040_sfe_v0.3.brd (EAGLE design)
At the start: 101.6 x 57.1 mm, 79 parts, among them IC2 93LC46ST, U2 TPD3E001DRLR, X1 332-12, X2 332-12, X3 52745-1690, X4 52745-1290

Commit message: Basic power planes and vias
Parts:
- added TP56, TP57, TP58, TP59, TP60, TP61, TP62, TP63, TP64, TP65: TPTP15SQ, testpad:TP15SQ
- added TP66, TP67, TP68, TP69: TPTP15R, testpad:TP15R
- added X5: 52745-2490, con-molex:52745-2490
- moved X4 111.7 mm to (8.26, 34.3), turned to 270 degrees
- flipped TP1 to the bottom
- flipped TP10 to the bottom
- flipped TP11 to the bottom
- flipped TP12 to the bottom
- flipped TP13 to the bottom
- flipped TP14 to the bottom
- flipped TP15 to the bottom
- flipped TP16 to the bottom
- flipped TP2 to the bottom
- flipped TP21 to the bottom
- flipped TP22 to the bottom
- flipped TP23 to the bottom
- flipped TP24 to the bottom
- flipped TP25 to the bottom
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Connections:
- net N$1 renamed VDD_DIG
- net N$2 renamed VREFP
- net N$3 renamed VSS_DIG
- net N$4 renamed AVDD_HV
- net N$65 renamed AVDD_LV
- net N$66 renamed AVSS_HV
- net N$67 renamed VDD_LVDS
- new net N$1: TP62.TP, U$1.D15
- new net N$2: TP61.TP, U$1.E15
- new net N$3: TP60.TP, U$1.D09
- new net N$4: TP59.TP, U$1.C09
- new net N$65: TP58.TP, U$1.D07
- new net N$66: TP57.TP, U$1.D06
- new net N$67: TP56.TP, U$1.D05
- new net N$84: TP63.TP, U$1.AA16
- new net N$85: TP65.TP, U$1.E09
- new net N$86: TP64.TP, U$1.AA09
- new net N$87: TP66.TP, U$1.AB09
- new net N$88: TP67.TP, U$1.E07
- new net N$89: TP68.TP, U$1.D08
- new net N$90: TP69.TP, U$1.AB08
Routing:
- net VSS_DIG: track 0.00 -> 41.0 mm, vias 0 -> 34
- net AVSS_HV: track 0.00 -> 5.39 mm, vias 0 -> 10
- net N$67: track 0.00 -> 0.90 mm, vias 0 -> 1
- net N$65: track 0.00 -> 0.90 mm, vias 0 -> 1
- net N$89: track 0.00 -> 0.90 mm, vias 0 -> 1
- net N$66: track 0.00 -> 0.90 mm, vias 0 -> 1
- net N$3: track 0.00 -> 0.90 mm, vias 0 -> 1
- added copper zone on layer 1, net AVDD_HV
- added copper zone on layer 1, net AVDD_LV
- added copper zone on layer 1, net AVSS_HV
- added copper zone on layer 16, net AVSS_HV
- added copper zone on layer 1, net VDD_DIG
- added copper zone on layer 1, net VDD_LVDS
- added copper zone on layer 1, net VREFP
- added copper zone on layer 1, net VSS_DIG

Commit message: Some minor updates
Parts:
- added U$3: IP4786CZ32SOT617-3, IP4786CZ32:SOT617-3
- moved CN1 7.65 mm to (92.1, 30.5)
- moved U$5 5.99 mm to (76.2, 37.5)
Connections:
- new net C_5V: U$3.13
- new net N$100: U$3.10, U$5.34
- new net N$101: U$3.32, U$5.16
- new net N$102: U$3.29, U$5.30
- new net N$103: CN1.13, U$3.25
- new net N$104: CN1.19, U$3.12
- new net N$105: CN1.16, U$3.14
- new net N$106: CN1.15, U$3.15
- new net N$107: CN1.3, U$3.23
- new net N$108: CN1.1, U$3.24
- new net N$109: CN1.6, U$3.21
- new net N$110: CN1.4, U$3.22
- new net N$111: CN1.9, U$3.19
- new net N$112: CN1.7, U$3.20
- new net N$113: CN1.12, U$3.17
- new net N$114: CN1.10, U$3.18
- new net N$115: U$5.45, U$5.46, U$5.47, U$5.48, U$5.49, U$5.50, U$5.52, U$5.54, U$5.55, U$5.56, U$5.57, U$5.58, U$5.59, U$5.60, U$5.61, U$5.62
- new net N$116: U$5.37, U$5.38, U$5.39, U$5.40, U$5.41, U$5.42, U$5.43, U$5.44
- new net N$91: U$3.7, U$5.18
- new net N$92: U$3.8, U$5.17
- new net N$93: U$3.5, U$5.21
- new net N$94: U$3.6, U$5.20
- new net N$95: U$3.3, U$5.24
- new net N$96: U$3.4, U$5.23
- new net N$97: U$3.1, U$5.27
- new net N$98: U$3.2, U$5.26
- new net N$99: U$3.9, U$5.33
- new net S_VCC: U$3.27
- new net VCC5V: U$3.11
- net EPAD: now also U$3.EPAD
